Commit message: update

File: modelo_sagan/urdf/modelo_sagan.urdf (robot description, URDF)
Before this commit: robot modelo_sagan, 7 links, 6 joints
Joints:
- removed joint eixo
- removed joint eixo1
- removed joint eixo2
- removed joint eixo3
- removed joint eixo4
- added joint eixoLBW: type fixed, parent Susp_left, child L_Back_wheel, origin xyz=0.000832348418708467 0.206985189270995 0 rpy=3.14159265358979 0 -0.835419970873937, axis 0 0 -1
- added joint eixoLFW: type fixed, parent Susp_left, child L_Front_wheel, origin xyz=-0.178838257906464 -0.104213429510898 -0.0204124999999994 rpy=3.14159265358979 0 -0.420787783674323, axis 0 0 0
- added joint eixoRBW: type fixed, parent Susp_right, child R_Back_wheel, origin xyz=-0.178838257906476 -0.104213429510882 -0.0483125 rpy=0 0 2.14187631042243, axis 0 0 0
- added joint eixoRFW: type fixed, parent Susp_right, child R_Front_wheel, origin xyz=0.00083235 0.20699 -0.050813 rpy=3.1416 0 -0.55205, axis 0 0 0
- added joint eixo_Susp_L: type fixed, parent base_link, child Susp_left, origin xyz=-0.0492787962347225 -0.1596 0.0314863650603519 rpy=-1.5707963267949 -1.0764644338619 3.14159265358979, axis 0 0 1
- joint eixo_Susp_R: type continuous -> fixed
